Commit message: Aggiunti due nodi: - Nodo test_Reachability: verifica se un punto nello spazio è raggiungibile dal robot tramite MoveIt. - Nodo build_scene: costruisce la scena di ostacoli leggendo la descrizione da file YAML e inserendo le mesh nel planning scene.

File: install/iiwa_description/share/iiwa_description/urdf/scene_obstacles.urdf.xacro (robot description, xacro)
@@ -183,5 +183,5 @@
     <link name="floor">
       <visual>
-        <origin xyz="1.0 0.5 0" rpy="${floor_roll} ${floor_pitch} ${floor_yaw}"/>
+        <origin xyz="0.0 0.0 0" rpy="${floor_roll} ${floor_pitch} ${floor_yaw}"/>
         <geometry>
           <mesh filename="file://$(find iiwa_description)/meshes/obstacles/Pavimento1.stl" scale ="0.001 0.001 0.001"/>
@@ -204,5 +204,5 @@
       <parent link="${parent}"/>
       <child link="floor"/>
-      <origin xyz="-2.25 -1.0 0.0" rpy="0 0 0"/>
+      <origin xyz="-1.25 -0.5 0.0" rpy="0 0 0"/>
     </joint>
   </xacro:macro>
