Commit message: Aggiunto package build_scene_package con il nodo build_scene_mesh per la descrizione e l'inserimento del collision object della cella. Inserito inoltre il nodo per il test di raggiungibilità del workspace tramite visualizzazione marker in RViz.

File: src/iiwa_config_moveit_config/config/urdf/dual_iiwa_robot.urdf.xacro (robot description, xacro)
@@ -1,23 +1,23 @@
 <?xml version="1.0"?>
 <robot xmlns:xacro="http://www.ros.org/wiki/xacro" name="dual_iiwa_robot">
-  <xacro:include filename="$(find iiwa_config)/config/urdf/dual_iiwa_robot.ros2_control.xacro" />
+  <xacro:include filename="$(find iiwa_config_moveit_config)/config/urdf/dual_iiwa_robot.ros2_control.xacro" />
   <xacro:include filename="$(find iiwa_description)/urdf/iiwa_arm_tcp.urdf.xacro" />
   <!-- Add ros2_control for dual arms -->
  <xacro:dual_iiwa_ros2_control name="iiwa" />
   <material name="gray">
-    <color rgba="0.5 0.5 0.5 1.0"/>
+    <color rgba="0.5 0.5 0.5 1"/>
   </material>
   <!-- Properties for the torso/base dimensions -->
   <xacro:property name="torso_width" value="0.30" />  <!-- 60cm wide -->
   <xacro:property name="torso_depth" value="0.30" />  <!-- 30cm deep -->
-  <xacro:property name="torso_height" value="1.0" /> <!-- 40cm high -->
-  <xacro:property name="shoulder_offset" value="0.15" /> <!-- Distance from center to shoulders -->
+  <xacro:property name="torso_height" value="0.92" /> <!-- 40cm high -->
+  <xacro:property name="shoulder_offset" value="0.176" /> <!-- Distance from center to shoulders -->
   <!-- Global robot translation: change these to move the whole robot in the world -->
   <xacro:property name="robot_x" value="-0.90" />
   <xacro:property name="robot_y" value="-0.43" />
-  <xacro:property name="robot_z" value="0.0" />
+  <xacro:property name="robot_z" value="0.462" />
   <!-- Materials -->
   <material name="torso_color">
-    <color rgba="0.7 0.7 0.8 0.5"/>
+    <color rgba="0.7 0.7 0.8 1"/>
   </material>
   <material name="mount_color">
@@ -32,18 +32,18 @@
   <link name="torso_base">
     <visual>
-      <origin xyz="0 0 ${torso_height/2}" rpy="0 0 0"/>
+      <origin xyz="0 0 0" rpy="1.57 0 0"/>
       <geometry>
-        <box size="${torso_depth} ${torso_width} ${torso_height}"/>
+      <mesh filename="file://$(find iiwa_description)/meshes/Busto.stl" scale="0.001 0.001 0.001"/>
       </geometry>
       <material name="torso_color"/>
     </visual>
     <collision>
-      <origin xyz="0 0 ${torso_height/2}" rpy="0 0 0"/>
+      <origin xyz="0 0 0" rpy="1.57 0 0"/>
       <geometry>
-        <box size="${torso_depth} ${torso_width} ${torso_height}"/>
+      <mesh filename="file://$(find iiwa_description)/meshes/Busto.stl" scale="0.001 0.001 0.001"/>
       </geometry>
     </collision>
     <inertial>
-      <origin xyz="0 0 ${torso_height/2}" rpy="0 0 0"/>
+      <origin xyz="0 0 0" rpy="1.57 0 0"/>
       <mass value="50.0"/>
       <inertia ixx="4.0" ixy="0.0" ixz="0.0" iyy="3.0" iyz="0.0" izz="2.0"/>
@@ -61,14 +61,9 @@
     <visual>
       <origin xyz="0 0 0" rpy="0 0 0"/>
-      <geometry>
-        <cylinder radius="0.05" length="0.1"/>
-      </geometry>
       <material name="mount_color"/>
     </visual>
     <collision>
       <origin xyz="0 0 0" rpy="0 0 0"/>
-      <geometry>
-        <cylinder radius="0.05" length="0.1"/>
-      </geometry>
+            <material name="mount_color"/>
     </collision>
     <inertial>
@@ -81,14 +76,9 @@
     <visual>
       <origin xyz="0 0 0" rpy="0 0 0"/>
-      <geometry>
-        <cylinder radius="0.05" length="0.1"/>
-      </geometry>
       <material name="mount_color"/>
     </visual>
     <collision>
       <origin xyz="0 0 0" rpy="0 0 0"/>
-      <geometry>
-        <cylinder radius="0.05" length="0.1"/>
-      </geometry>
+      <material name="mount_color"/>
     </collision>
     <inertial>
@@ -102,5 +92,5 @@
     <child link="left_shoulder_mount"/>
     <!-- Left shoulder: ruotato di 90 gradi attorno Y per essere orizzontale, poi 90 attorno Z per puntare a sinistra -->
-    <origin xyz="0 ${shoulder_offset} ${torso_height}" rpy="0 ${pi/2 - 11.3*pi/180} ${pi/2}"/>
+    <origin xyz="0 ${shoulder_offset} 0.402" rpy="0 ${pi/2 - 11.3*pi/180} ${pi/2}"/>
   </joint>
   <!-- Joint connecting torso to right shoulder mount -->
@@ -109,5 +99,5 @@
     <child link="right_shoulder_mount"/>
     <!-- Right shoulder: ruotato di 90 gradi attorno Y per essere orizzontale, poi -90 attorno Z per puntare a destra -->
-    <origin xyz="0 ${-shoulder_offset} ${torso_height}" rpy="0 ${pi/2 - 11.3*pi/180} ${-pi/2}"/>
+    <origin xyz="0 ${-shoulder_offset} 0.402" rpy="0 ${pi/2 - 11.3*pi/180} ${-pi/2}"/>
   </joint>
   <!-- Left IIWA arm -->

File: src/iiwa_description/urdf/dual_iiwa_robot.urdf.xacro (robot description, xacro)
@@ -1,23 +1,23 @@
 <?xml version="1.0"?>
 <robot xmlns:xacro="http://www.ros.org/wiki/xacro" name="dual_iiwa_robot">
-  <xacro:include filename="$(find iiwa_config)/config/urdf/dual_iiwa_robot.ros2_control.xacro" />
+  <xacro:include filename="$(find iiwa_config_moveit_config)/config/urdf/dual_iiwa_robot.ros2_control.xacro" />
   <xacro:include filename="$(find iiwa_description)/urdf/iiwa_arm_tcp.urdf.xacro" />
   <!-- Add ros2_control for dual arms -->
- <!--- <xacro:dual_iiwa_ros2_control name="iiwa" />-->
+  <xacro:dual_iiwa_ros2_control name="iiwa" />
   <material name="gray">
-    <color rgba="0.5 0.5 0.5 1.0"/>
+    <color rgba="0.5 0.5 0.5 1"/>
   </material>
   <!-- Properties for the torso/base dimensions -->
   <xacro:property name="torso_width" value="0.30" />  <!-- 60cm wide -->
   <xacro:property name="torso_depth" value="0.30" />  <!-- 30cm deep -->
-  <xacro:property name="torso_height" value="1.0" /> <!-- 40cm high -->
-  <xacro:property name="shoulder_offset" value="0.15" /> <!-- Distance from center to shoulders -->
+  <xacro:property name="torso_height" value="0.92" /> <!-- 40cm high -->
+  <xacro:property name="shoulder_offset" value="0.176" /> <!-- Distance from center to shoulders -->
   <!-- Global robot translation: change these to move the whole robot in the world -->
   <xacro:property name="robot_x" value="-0.90" />
   <xacro:property name="robot_y" value="-0.43" />
-  <xacro:property name="robot_z" value="0.0" />
+  <xacro:property name="robot_z" value="0.462" />
   <!-- Materials -->
   <material name="torso_color">
-    <color rgba="0.7 0.7 0.8 0.5"/>
+    <color rgba="0.7 0.7 0.8 1"/>
   </material>
   <material name="mount_color">
@@ -32,18 +32,18 @@
   <link name="torso_base">
     <visual>
-      <origin xyz="0 0 ${torso_height/2}" rpy="0 0 0"/>
+      <origin xyz="0 0 0" rpy="1.57 0 0"/>
       <geometry>
-        <box size="${torso_depth} ${torso_width} ${torso_height}"/>
+      <mesh filename="file://$(find iiwa_description)/meshes/Busto.stl" scale="0.001 0.001 0.001"/>
       </geometry>
       <material name="torso_color"/>
     </visual>
     <collision>
-      <origin xyz="0 0 ${torso_height/2}" rpy="0 0 0"/>
+      <origin xyz="0 0 0" rpy="1.57 0 0"/>
       <geometry>
-        <box size="${torso_depth} ${torso_width} ${torso_height}"/>
+      <mesh filename="file://$(find iiwa_description)/meshes/Busto.stl" scale="0.001 0.001 0.001"/>
       </geometry>
     </collision>
     <inertial>
-      <origin xyz="0 0 ${torso_height/2}" rpy="0 0 0"/>
+      <origin xyz="0 0 0" rpy="1.57 0 0"/>
       <mass value="50.0"/>
       <inertia ixx="4.0" ixy="0.0" ixz="0.0" iyy="3.0" iyz="0.0" izz="2.0"/>
@@ -61,7 +61,4 @@
     <visual>
       <origin xyz="0 0 0" rpy="0 0 0"/>
-      <geometry>
-        <cylinder radius="0.05" length="0.1"/>
-      </geometry>
       <material name="mount_color"/>
     </visual>
@@ -102,5 +99,5 @@
     <child link="left_shoulder_mount"/>
     <!-- Left shoulder: ruotato di 90 gradi attorno Y per essere orizzontale, poi 90 attorno Z per puntare a sinistra -->
-    <origin xyz="0 ${shoulder_offset} ${torso_height}" rpy="0 ${pi/2 - 11.3*pi/180} ${pi/2}"/>
+    <origin xyz="0 ${shoulder_offset} 0.402" rpy="0 ${pi/2 - 11.3*pi/180} ${pi/2}"/>
   </joint>
   <!-- Joint connecting torso to right shoulder mount -->
@@ -109,5 +106,5 @@
     <child link="right_shoulder_mount"/>
     <!-- Right shoulder: ruotato di 90 gradi attorno Y per essere orizzontale, poi -90 attorno Z per puntare a destra -->
-    <origin xyz="0 ${-shoulder_offset} ${torso_height}" rpy="0 ${pi/2 - 11.3*pi/180} ${-pi/2}"/>
+    <origin xyz="0 ${-shoulder_offset} 0.402" rpy="0 ${pi/2 - 11.3*pi/180} ${-pi/2}"/>
   </joint>
   <!-- Left IIWA arm -->
@@ -119,4 +116,3 @@
     <origin xyz="0 0 0" rpy="0 0 0"/>
   </xacro:iiwa_arm_tcp>
- <!--  <xacro:scene_obstacles parent="world"/>-->
 </robot>

File: src/iiwa_description/urdf/iiwa_arm_tcp.urdf.xacro (robot description, xacro)
@@ -7,14 +7,15 @@
     </xacro:iiwa_arm>
 <!--Ora dobbiamo aggiungere il tcp-->
- <link name="${prefix}tcp">
+ <link name="${prefix}hand">
     <visual>
-      <origin xyz="0 0 0" rpy="0 0 0"/>
+      <origin xyz="0 0 0" rpy="0 0 0.0"/>
       <geometry>
         <!-- SCHUNK end-effector mesh (file present in meshes/) -->
           <mesh filename="file://$(find iiwa_description)/meshes/schunk.stl" scale ="0.001 0.001 0.001"/>
       </geometry>
+      <material name="gray"/>
     </visual>
     <collision>
-      <origin xyz="0 0 0" rpy="0 0 0"/>
+      <origin xyz="0 0 0" rpy="0 0 0.0"/>
       <geometry>
           <mesh filename="file://$(find iiwa_description)/meshes/schunk.stl" scale ="0.001 0.001 0.001"/>
@@ -22,31 +23,31 @@
     </collision>
     <inertial>
-      <origin xyz="0 0 0" rpy="0 0 0"/>
+      <origin xyz="0 0 0" rpy="0 0 0.0"/>
       <mass value="0.5"/>
       <inertia ixx="0.0" ixy="0.0" ixz="0.0" iyy="0.0" iyz="0.0" izz="0.0"/>
     </inertial>
   </link>
-  <joint name="${prefix}tool0_to_tcp" type="fixed">
-    <origin rpy="1.57 0 0" xyz="0 -0.05 0"/>
+  <joint name="${prefix}tool0_to_hand" type="fixed">
+    <origin rpy="0 0 0" xyz="0 0.0 0.06"/>
     <parent link="${prefix}tool0"/>
-    <child link="${prefix}tcp"/>
+    <child link="${prefix}hand"/>
   </joint>
- <link name="${prefix}finger_left">
+<link name="${prefix}finger_left">
+     <material name="gray"/>
     <visual>
-      <!-- finger is a thin rectangular box; tune size as needed -->
-      <origin xyz="0 0 0" rpy="0 0 0"/>
-      <geometry>
-        <box size="0.02 0.08 0.02"/> <!-- x(width) y(thickness) z(length) -->
+      <origin xyz="0 0 0" rpy="0 0 1.57"/>
+    <geometry>
+          <mesh filename="file://$(find iiwa_description)/meshes/finger.stl" scale ="0.001 0.001 0.001"/>
       </geometry>
-        <color rgba="1 0.58 0.66 1"/>
+      <material name="gray"/>
     </visual>
     <collision>
-      <origin xyz="0 0 0" rpy="0 0 0"/>
+      <origin xyz="0 0 0" rpy="0 0 1.57"/>
       <geometry>
-        <box size="0.02 0.08 0.02"/>
+          <mesh filename="file://$(find iiwa_description)/meshes/finger.stl" scale ="0.001 0.001 0.001"/>
       </geometry>
     </collision>
     <inertial>
-      <origin xyz="0 0 0" rpy="0 0 0"/>
+      <origin xyz="0 0 0" rpy="0 0 1.57"/>
       <mass value="0.05"/>
       <inertia ixx="0.0001" ixy="0" ixz="0" iyy="0.0001" iyz="0" izz="0.0001"/>
@@ -54,36 +55,47 @@
   </link>
   <link name="${prefix}finger_right">
-     <material name="gray"/>
     <visual>
-      <origin xyz="0 0 0" rpy="0 0 0"/>
-      <geometry>
-        <box size="0.02 0.08 0.02"/>
+      <origin xyz="0 0 0" rpy="0 0 1.57"/>
+    <geometry>
+          <mesh filename="file://$(find iiwa_description)/meshes/finger.stl" scale ="0.001 0.001 0.001"/>
       </geometry>
+           <material name="gray"/>
     </visual>
     <collision>
-      <origin xyz="0 0 0" rpy="0 0 0"/>
+      <origin xyz="0 0 0" rpy="0 0 1.57"/>
       <geometry>
-        <box size="0.02 0.08 0.02"/>
+          <mesh filename="file://$(find iiwa_description)/meshes/finger.stl" scale ="0.001 0.001 0.001"/>
       </geometry>
     </collision>
     <inertial>
-      <origin xyz="0 0 0" rpy="0 0 0"/>
+      <origin xyz="0 0 0" rpy="0 0 1.57"/>
       <mass value="0.05"/>
       <inertia ixx="0.0001" ixy="0" ixz="0" iyy="0.0001" iyz="0" izz="0.0001"/>
     </inertial>
   </link>
-  <joint name="${prefix}tcp_to_finger_left" type="prismatic">
-    <origin xyz="0.01 0.12 -0.1" rpy="0 0 0"/>
-    <parent link="${prefix}tcp"/>
+  <joint name="${prefix}hand_to_finger_left" type="prismatic">
+    <origin xyz="0.017 0.064 0.10" rpy="0 0 0"/>
+    <parent link="${prefix}hand"/>
     <child link="${prefix}finger_left"/>
-      <axis xyz="0 0 -1" />
-        <limit effort="20" lower="0.0" upper="0.04" velocity="0.2" />
+      <axis xyz="0 -1 0" />
+        <limit effort="20" lower="0.02" upper="0.00" velocity="0.2" />
   </joint>
-  <joint name="${prefix}tcp_to_finger_right" type="prismatic">
-    <origin xyz="0.01 0.12 0.0" rpy="0 0 0"/>
-    <parent link="${prefix}tcp"/>
+  <joint name="${prefix}hand_to_finger_right" type="prismatic">
+    <origin xyz="0.016 -0.042 0.10" rpy="0 0 0"/>
+    <parent link="${prefix}hand"/>
     <child link="${prefix}finger_right"/>
-      <axis xyz="0 0 -1" />
-        <limit effort="20" lower="0.0" upper="0.04" velocity="0.2" />
+      <axis xyz="0 1 0" />
+        <limit effort="20" lower="0.0" upper="0.02" velocity="0.2" />
+  </joint>
+  <link name="${prefix}tcp">
+    <visual>
+      <origin xyz="0 0 0" rpy="0 0 0"/>
+      <material name="blue"/>
+    </visual>
+   </link>
+   <joint name="${prefix}hand_to_tcp" type="fixed">
+    <origin rpy="0 0 0" xyz="0 0.0 0.12"/>
+    <parent link="${prefix}hand"/>
+    <child link="${prefix}tcp"/>
   </joint>
 </xacro:macro>

File: src/iiwa_description/urdf/scene_environment.urdf.xacro (robot description, xacro)
@@ -2,8 +2,8 @@
 <robot xmlns:xacro="http://www.ros.org/wiki/xacro" name="scene_environment">
   <!-- Include the scene obstacles -->
-  <xacro:include filename="$(find iiwa_description)/urdf/scene_obstacles.urdf.xacro" />
+  <xacro:include filename="$(find iiwa_description)/urdf/scene_total_evironment.urdf.xacro" />
   <!-- Base/World link for the environment -->
   <link name="world"/>
   <!-- Include scene obstacles -->
-  <xacro:scene_obstacles parent="world"/>
+  <xacro:scene_total_evironment parent="world"/>
 </robot>

File: src/iiwa_description/urdf/scene_obstacles.urdf.xacro (robot description, xacro)
@@ -53,5 +53,30 @@
     <parent link="${parent}"/>
     <child link="frigorifero"/>
-    <origin xyz="1.87 2.0 0.0" rpy="0 0 0"/>
+    <origin xyz="1.87 2.62 0.0" rpy="0 0 0"/>
+  </joint>
+  <link name="Congelatore">
+    <visual>
+      <origin xyz="0 0 0" rpy="1.57 0 3.14"/>
+      <geometry>
+        <mesh filename="file://$(find iiwa_description)/meshes/obstacles/Congelatore.stl" scale="0.001 0.001 0.001"/>
+      </geometry>
+      <material name="table_color"/>
+    </visual>
+    <collision>
+      <origin xyz="0 0 0" rpy="1.57 0 3.14"/>
+      <geometry>
+        <mesh filename="file://$(find iiwa_description)/meshes/obstacles/Congelatore.stl" scale="0.001 0.001 0.001"/>
+      </geometry>
+    </collision>
+    <inertial>
+      <origin xyz="0 0 0" rpy="1.57 0 3.14"/>
+      <mass value="30.0"/>
+      <inertia ixx="5.0" ixy="0.0" ixz="0.0" iyy="5.0" iyz="0.0" izz="5.0"/>
+    </inertial>
+  </link>
+  <joint name="world_to_Congelatore" type="fixed">
+    <parent link="${parent}"/>
+    <child link="Congelatore"/>
+    <origin xyz="1.87 1.85 0.0" rpy="0 0 0"/>
   </joint>
   <link name="Roboqbo">
@@ -78,5 +103,5 @@
     <parent link="${parent}"/>
     <child link="Roboqbo"/>
-    <origin xyz="-1.60 -0.32 0.0" rpy="0 0 0"/>
+    <origin xyz="-1.60 -0.32 0.07" rpy="0 0 0"/>
   </joint>
     <link name="Rastrelliera">
@@ -103,5 +128,30 @@
     <parent link="${parent}"/>
     <child link="Rastrelliera"/>
-    <origin xyz="-0.28 -0.11 0.86" rpy="0 0 0"/>
+    <origin xyz="-0.26 -0.11 0.86" rpy="0 0 0"/>
+  </joint>
+ <link name="Deimpilatore_piatti">
+    <visual>
+      <origin xyz="0 0 0" rpy="1.57 3.14 0"/>
+      <geometry>
+        <mesh filename="file://$(find iiwa_description)/meshes/obstacles/Deimpilatore_piatti.stl" scale="0.001 0.001 0.001"/>
+      </geometry>
+      <material name="table_color"/>
+    </visual>
+    <collision>
+      <origin xyz="0 0 0" rpy="1.57 3.14 0"/>
+      <geometry>
+        <mesh filename="file://$(find iiwa_description)/meshes/obstacles/Deimpilatore_piatti.stl" scale="0.001 0.001 0.001"/>
+      </geometry>
+    </collision>
+    <inertial>
+      <origin xyz="0 0 0" rpy="1.57 3.14 0"/>
+      <mass value="30.0"/>
+      <inertia ixx="5.0" ixy="0.0" ixz="0.0" iyy="5.0" iyz="0.0" izz="5.0"/>
+    </inertial>
+  </link>
+  <joint name="world_to_Deimpilatore_piatti" type="fixed">
+    <parent link="${parent}"/>
+    <child link="Deimpilatore_piatti"/>
+    <origin xyz="-0.20 -1.08 1.80" rpy="0 0 0"/>
   </joint>
      <link name="Trasportatore1">
@@ -153,5 +203,5 @@
     <parent link="${parent}"/>
     <child link="Tavolo_inox"/>
-    <origin xyz="0.0 0.41 0.842" rpy="0 0 0"/>
+    <origin xyz="0.02 0.41 0.842" rpy="0 0 0"/>
   </joint>
      <link name="Tavolo_inox2">
@@ -178,5 +228,5 @@
     <parent link="${parent}"/>
     <child link="Tavolo_inox2"/>
-    <origin xyz="-0.675 1.26 0.842" rpy="0 0 0"/>
+    <origin xyz="-0.680 1.24 0.842" rpy="0 0 0"/>
   </joint>
     <!-- Floor -->

Commit message: Versione definitiva corretta

File: src/iiwa_config_moveit_config/config/urdf/dual_iiwa_robot.urdf.xacro (robot description, xacro)
@@ -18,5 +18,5 @@
   <xacro:property name="robot_x" value="-0.90" />
   <xacro:property name="robot_y" value="-0.43" />
-  <xacro:property name="robot_z" value="0.462" />
+  <xacro:property name="robot_z" value="0.489" />
   <!-- Materials -->
   <material name="torso_color">

File: src/iiwa_config_moveit_config/config/urdf/dual_iiwa_robot_hand.ros2_control.xacro (robot description, xacro)
@@ -8,10 +8,6 @@
       <joint name="left_hand_to_finger_left">
         <command_interface name="position"/>
-        <state_interface name="position">
-          <param name="initial_value" value="0.0"/>
-        </state_interface>
-        <state_interface name="velocity">
-          <param name="initial_value" value="0.0"/>
-        </state_interface>
+        <state_interface name="position"/>
+        <state_interface name="velocity"/>
       </joint>
       <joint name="left_hand_to_finger_right">
@@ -26,10 +22,6 @@
       <joint name="right_hand_to_finger_left">
         <command_interface name="position"/>
-        <state_interface name="position">
-          <param name="initial_value" value="0.0"/>
-        </state_interface>
-        <state_interface name="velocity">
-          <param name="initial_value" value="0.0"/>
-        </state_interface>
+        <state_interface name="position"/>
+        <state_interface name="velocity"/>
       </joint>
       <joint name="right_hand_to_finger_right">

File: src/iiwa_description/urdf/iiwa_arm_tcp.urdf.xacro (robot description, xacro)
@@ -19,5 +19,5 @@
       <origin xyz="0 0 0" rpy="0 0 0.0"/>
       <geometry>
-          <mesh filename="file://$(find iiwa_description)/meshes/schunk.stl" scale ="0.001 0.001 0.001"/>
+          <mesh filename="file://$(find iiwa_description)/meshes/bounding_primitive_hand.stl" scale ="0.001 0.001 0.001"/>
       </geometry>
     </collision>
@@ -36,14 +36,15 @@
      <material name="gray"/>
     <visual>
-      <origin xyz="0 0 0" rpy="0 0 1.57"/>
+      <origin xyz="0 0 0.0" rpy="0 0 1.57"/>
     <geometry>
-          <mesh filename="file://$(find iiwa_description)/meshes/finger.stl" scale ="0.001 0.001 0.001"/>
+           <mesh filename="file://$(find iiwa_description)/meshes/finger_left.stl" scale ="0.001 0.001 0.001"/>
       </geometry>
       <material name="gray"/>
     </visual>
     <collision>
-      <origin xyz="0 0 0" rpy="0 0 1.57"/>
+      <origin xyz="0 0 0.0" rpy="0 0 1.57"/>
       <geometry>
-          <mesh filename="file://$(find iiwa_description)/meshes/finger.stl" scale ="0.001 0.001 0.001"/>
+          <!-- Box semplice invece di mesh per collision più preciso -->
+            <box size="0.026 0.02 0.13"/>
       </geometry>
     </collision>
@@ -56,14 +57,15 @@
   <link name="${prefix}finger_right">
     <visual>
-      <origin xyz="0 0 0" rpy="0 0 1.57"/>
+      <origin xyz="0 0 0.00" rpy="0 0 1.57"/>
     <geometry>
-          <mesh filename="file://$(find iiwa_description)/meshes/finger.stl" scale ="0.001 0.001 0.001"/>
+            <mesh filename="file://$(find iiwa_description)/meshes/finger_right.stl" scale ="0.001 0.001 0.001"/>
       </geometry>
            <material name="gray"/>
     </visual>
     <collision>
-      <origin xyz="0 0 0" rpy="0 0 1.57"/>
+      <origin xyz="0 0 0.0" rpy="0 0 0"/>
       <geometry>
-          <mesh filename="file://$(find iiwa_description)/meshes/finger.stl" scale ="0.001 0.001 0.001"/>
+          <!-- Box semplice invece di mesh per collision più preciso -->
+            <box size="0.026 0.02 0.13"/>
       </geometry>
     </collision>
@@ -75,5 +77,5 @@
   </link>
   <joint name="${prefix}hand_to_finger_left" type="prismatic">
-    <origin xyz="0.017 0.064 0.10" rpy="0 0 0"/>
+    <origin xyz="0.017 0.042 0.10" rpy="0 0 0"/>
     <parent link="${prefix}hand"/>
     <child link="${prefix}finger_left"/>
@@ -82,5 +84,5 @@
   </joint>
   <joint name="${prefix}hand_to_finger_right" type="prismatic">
-    <origin xyz="0.016 -0.042 0.10" rpy="0 0 0"/>
+    <origin xyz="0.017 -0.042 0.10" rpy="0 0 0"/>
     <parent link="${prefix}hand"/>
     <child link="${prefix}finger_right"/>

File: src/iiwa_description/urdf/scene_environment.urdf.xacro (robot description, xacro)
@@ -2,8 +2,8 @@
 <robot xmlns:xacro="http://www.ros.org/wiki/xacro" name="scene_environment">
   <!-- Include the scene obstacles -->
-  <xacro:include filename="$(find iiwa_description)/urdf/scene_total_evironment.urdf.xacro" />
+  <xacro:include filename="$(find iiwa_description)/urdf/scene_obstacles.urdf.xacro" />
   <!-- Base/World link for the environment -->
   <link name="world"/>
   <!-- Include scene obstacles -->
-  <xacro:scene_total_evironment parent="world"/>
+  <xacro:scene_obstacles parent="world"/>
 </robot>

File: src/iiwa_description/urdf/scene_obstacles.urdf.xacro (robot description, xacro)
@@ -6,9 +6,6 @@
     <xacro:property name="floor_pitch" value="0.0" />
     <xacro:property name="floor_yaw" value="1.57" />
-  <!-- adjust joint z to translate the floor in world coordinates if needed -->
   <xacro:property name="floor_z_offset" value="0.0" />
-  <!-- visual offset: use this to shift the mesh relative to the floor link frame (to center it) -->
   <xacro:property name="floor_visual_xyz" value="-0.5 0 0" />
-    <!-- Materials for obstacles  qui vado a inizializzare ostacoli con colori -->
     <material name="table_color">
 <color rgba="0.2 0.2 0.2 1.0"/>
@@ -257,3 +254,3 @@
     </joint>
   </xacro:macro>
-</robot>
+</robot>  <xacro:property name="floor_z_offset" value="0.0" />
